File: hardware/controller.sch (EAGLE design)
At the start: 18 parts, among them J4 AVR_SPI_PROG_3X2PTH, U1 ATMEGA328P-AU, U2 MAX6675

Commit message: layout done
Parts:
- added J6: (no value), SparkFun-Connectors:CONN_02PTH3
Connections:
- new net N$3: J6.2, U2.T-
- new net N$4: J6.1, U2.T+
Changed lines of the file:
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@@
 <part name="R4" library="passives-7351" deviceset="RESISTOR" device="0603-N" value="4k7"/>
 <part name="SUPPLY8" library="SparkFun-PowerSymbols" deviceset="VCC" device=""/>
+<part name="J6" library="SparkFun-Connectors" deviceset="CONN_02" device="PTH3"/>
 </parts>
 <sheets>
@@
 <instance part="R4" gate="G$1" x="111.76" y="30.48" rot="R90"/>
 <instance part="SUPPLY8" gate="G$1" x="111.76" y="35.56" smashed="yes"/>
+<instance part="J6" gate="G$1" x="73.66" y="5.08"/>
 </instances>
 <busses>
@@
 </segment>
 </net>
+<net name="N$3" class="0">
+<segment>
+<pinref part="U2" gate="G$1" pin="T-"/>
+<pinref part="J6" gate="G$1" pin="2"/>
+<wire x1="83.82" y1="7.62" x2="81.28" y2="7.62" width="0.1524" layer="91"/>
+</segment>
+</net>
+<net name="N$4" class="0">
+<segment>
+<pinref part="U2" gate="G$1" pin="T+"/>
+<pinref part="J6" gate="G$1" pin="1"/>
+<wire x1="83.82" y1="5.08" x2="81.28" y2="5.08" width="0.1524" layer="91"/>
+</segment>
+</net>
